File: board/bleriot-reg6.kicad_pcb (KiCad board)
At the start: 2 copper layers, 306 x 15.5 mm, 85 parts, among them J1 POWER, U1 LM358, U2 LM358, U3 LM358, U4 LM1117MP-3.3, U5 PY32F030F1xPx, U6 PAN2110P0AA, X1 SWD, Y1 16MHz

Commit message: Update Bleriot board files with footprint and clearance adjustments
- Modified copper edge clearance values in `bleriot-reg6.kicad_pro` to correct DRC exclusions.
- Changed footprint for a connector in `bleriot-reg6.kicad_sch` from Phoenix MC to MSTB series.
- Updated UUIDs and adjusted dimensions for pads and lines in `ssr-contact.kicad_mod` to enhance layout accuracy.
Parts:
- J1: footprint Connector_Phoenix_MC:PhoenixContact_MC_1,5_2-G-3.5_1x02_P3.50mm_Horizontal -> Connector_Phoenix_MSTB:PhoenixContact_MSTBA_2,5_2-G_1x02_P5.00mm_Horizontal
- moved A1 4.00 mm to (367.5, 144.6)
- moved C5 4.00 mm to (354.5, 150.0)
- moved C7 4.00 mm to (358.5, 150.0)
- moved U6 4.00 mm to (363.0, 146.5)
- moved Y1 4.00 mm to (357.5, 144.0)
- moved J1 3.95 mm to (68.0, 144.5)
- moved RE1 2.50 mm to (86.0, 141.5)
- moved RE6 2.50 mm to (346.0, 141.5)
- moved RE2 1.50 mm to (138.0, 141.5)
- moved RE5 1.50 mm to (294.0, 141.5)
- moved RE3 0.50 mm to (190.0, 141.5)
- moved RE4 0.50 mm to (242.0, 141.5)
Routing:
- net Net-(J1-Pin_2): track 16.2 -> 20.5 mm
- net /~{RF_CS}: track 100.6 -> 104.6 mm
- net /RF_DATA: track 92.5 -> 96.5 mm
- net /RF_SCK: track 94.1 -> 98.1 mm
- net +3V3: track 350.5 -> 354.5 mm
- net /channel-5/OPA_OUT: track 29.4 -> 26.7 mm
- net /channel-6/OPA_OUT: track 43.6 -> 46.3 mm
- net GND: vias 271 -> 269
Other:
- board size 306 x 15.5 mm -> 314 x 15.5 mm
- board text added: "reg6 v1.1"
- board text removed: "POWER"
- board text removed: "reg6 v1.0"
