File: board/bleriot-reg6.kicad_sch (KiCad schematic)
At the start: 25 parts, among them J1 POWER, U1 LM358, U2 LM358, U3 LM358, U4 LM1117MP-3.3, U5 PY32F030F1xPx, U6 PAN2110P0AA, X1 SWD, Y1 16MHz

Commit message: Update Bleriot board files with footprint and clearance adjustments
- Modified copper edge clearance values in `bleriot-reg6.kicad_pro` to correct DRC exclusions.
- Changed footprint for a connector in `bleriot-reg6.kicad_sch` from Phoenix MC to MSTB series.
- Updated UUIDs and adjusted dimensions for pads and lines in `ssr-contact.kicad_mod` to enhance layout accuracy.
Parts:
- J1: footprint Connector_Phoenix_MC:PhoenixContact_MC_1,5_2-G-3.5_1x02_P3.50mm_Horizontal -> Connector_Phoenix_MSTB:PhoenixContact_MSTBA_2,5_2-G_1x02_P5.00mm_Horizontal
Changed lines of the file:
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@@
 			)
 		)
-		(property "Footprint" "Connector_Phoenix_MC:PhoenixContact_MC_1,5_2-G-3.5_1x02_P3.50mm_Horizontal"
+		(property "Footprint" "Connector_Phoenix_MSTB:PhoenixContact_MSTBA_2,5_2-G_1x02_P5.00mm_Horizontal"
 			(at 105.41 171.45 0)
 			(hide yes)
